Commit message: urdf right and left track

File: track/robot.urdf (robot description, URDF)
Before this commit: robot track, 6 links, 5 joints
Links:
- removed link body
- added link body_left, mass 0.6; collision mesh filename=package://assets/body_left.stl; visual mesh filename=package://assets/body_left.stl
- added link body_right, mass 0.6; collision mesh filename=package://assets/body_right.stl; visual mesh filename=package://assets/body_right.stl
- added link wheel_5, mass 0.1; collision mesh filename=package://assets/wheel.stl; visual mesh filename=package://assets/wheel.stl
- added link wheel_6, mass 0.1; collision mesh filename=package://assets/wheel.stl; visual mesh filename=package://assets/wheel.stl
- added link wheel_7, mass 0.1; collision mesh filename=package://assets/wheel.stl; visual mesh filename=package://assets/wheel.stl
- added link wheel_8, mass 0.1; collision mesh filename=package://assets/wheel.stl; visual mesh filename=package://assets/wheel.stl
Joints:
- removed joint track
- removed joint wheel_1
- removed joint wheel_2
- removed joint wheel_3
- removed joint wheel_4
- added joint base_left: type revolute, parent body_left, child leg, origin xyz=-0.129266 -0.0575005 -0.0715997 rpy=1.5708 -6.45781e-16 -1.5708, axis 0 0 1, limit lower=-0.785398 upper=0.785398 effort=10 velocity=10
- added joint base_right: type revolute, parent leg, child body_right, origin xyz=-1.11022e-16 0 -0.06 rpy=-1.33599e-16 -7.87523e-16 -6.45781e-16, axis 0 0 1, limit lower=-0.785398 upper=0.785398 effort=10 velocity=10
- added joint wheel_1_left: type continuous, parent body_left, child wheel, origin xyz=-0.119266 -0.00909429 -0.129979 rpy=1.5708 6.42791e-09 1.5708, axis 0 0 1, limit effort=10 velocity=10
- added joint wheel_1_right: type continuous, parent body_right, child wheel_5, origin xyz=0.0766777 -0.0417374 0.01 rpy=-2.40478e-15 -1.41754e-14 -3.14159, axis 0 0 1, limit effort=10 velocity=10
- added joint wheel_2_left: type continuous, parent body_left, child wheel_2, origin xyz=-0.119266 -0.0575005 -0.129979 rpy=1.5708 0.0242209 1.5708, axis 0 0 1, limit effort=10 velocity=10
- added joint wheel_2_right: type continuous, parent body_right, child wheel_6, origin xyz=0.0510312 -0.0583795 0.01 rpy=-2.40478e-15 -1.41754e-14 -3.14159, axis 0 0 1, limit effort=10 velocity=10
- added joint wheel_3_left: type continuous, parent body_left, child wheel_3, origin xyz=-0.119266 -0.108532 -0.129979 rpy=1.5708 0.0242209 1.5708, axis 0 0 1, limit effort=10 velocity=10
- added joint wheel_3_right: type continuous, parent body_right, child wheel_7, origin xyz=-1.11022e-16 -0.0583795 0.01 rpy=-2.40478e-15 -1.41754e-14 -3.14159, axis 0 0 1, limit effort=10 velocity=10
- added joint wheel_4_left: type continuous, parent body_left, child wheel_4, origin xyz=-0.119266 -0.134178 -0.113337 rpy=1.5708 6.4279e-09 1.5708, axis 0 0 1, limit effort=10 velocity=10
- added joint wheel_4_right: type continuous, parent body_right, child wheel_8, origin xyz=-0.0484063 -0.0583795 0.01 rpy=-2.40478e-15 -1.41754e-14 -3.14159, axis 0 0 1, limit effort=10 velocity=10
