Commit message: trackquad urdf with track

File: track_left/robot.urdf (robot description, URDF)
Before this commit: robot track_left, 5 links, 4 joints
Joints:
- removed joint wheel_1_left
- removed joint wheel_2_left
- removed joint wheel_3_left
- removed joint wheel_4_left
- added joint wheel_1: type continuous, parent body_left, child wheel, origin xyz=0 0.0484063 -0.0583795 rpy=-6.12323e-17 -1.5708 0, axis 0 0 1, limit effort=10 velocity=10
- added joint wheel_2: type continuous, parent body_left, child wheel_2, origin xyz=0 1.07779e-16 -0.0583795 rpy=-6.12323e-17 -1.5708 0, axis 0 0 1, limit effort=10 velocity=10
- added joint wheel_3: type continuous, parent body_left, child wheel_3, origin xyz=0 -0.0510313 -0.0583795 rpy=-6.12323e-17 -1.5708 0, axis 0 0 1, limit effort=10 velocity=10
- added joint wheel_4: type continuous, parent body_left, child wheel_4, origin xyz=0 -0.0766777 -0.0417374 rpy=-6.12323e-17 -1.5708 0, axis 0 0 1, limit effort=10 velocity=10

File: track_right/robot.urdf (robot description, URDF)
Before this commit: robot track_right, 5 links, 4 joints
Joints:
- removed joint wheel_1
- removed joint wheel_2
- removed joint wheel_3
- removed joint wheel_4
- added joint wheel_1_left: type continuous, parent body_right, child wheel, origin xyz=2.08167e-17 0.0583795 0.0484062 rpy=-1.5708 0.992087 -1.5708, axis 0 0 1, limit effort=10 velocity=10
- added joint wheel_2_left: type continuous, parent body_right, child wheel_2, origin xyz=0 0.0583795 1.10544e-16 rpy=-1.5708 0.967866 -1.5708, axis 0 0 1, limit effort=10 velocity=10
- added joint wheel_3_left: type continuous, parent body_right, child wheel_3, origin xyz=-2.08167e-17 0.0583795 -0.0510312 rpy=-1.5708 0.967866 -1.5708, axis 0 0 1, limit effort=10 velocity=10
- added joint wheel_4_left: type continuous, parent body_right, child wheel_4, origin xyz=-3.46945e-17 0.0417374 -0.0766777 rpy=-1.5708 0.992087 -1.5708, axis 0 0 1, limit effort=10 velocity=10
