Commit message: change file to package

File: traquad/traquad/urdf/mulinex_little_with_track.urdf (robot description, URDF)
Before this commit: robot mulinex, 29 links, 28 joints
Links:
- link LF_SHOULDER: geometry collision box size=0.269 0.057 0.060; visual mesh filename=package://assets/Module_left_front.stl
- link LF_UPPER_LEG: geometry collision box size=0.269 0.057 0.060; visual mesh filename=package://assets/Module_left_front.stl
- link LH_SHOULDER: geometry collision box size=0.269 0.057 0.060; visual mesh filename=package://assets/Module_left_hind.stl
- link LH_UPPER_LEG: geometry collision box size=0.269 0.057 0.060; visual mesh filename=package://assets/Module_left_hind.stl
- link RF_SHOULDER: geometry collision box size=0.269 0.057 0.060; visual mesh filename=package://assets/Module_right_front.stl
- link RF_UPPER_LEG: geometry collision box size=0.269 0.057 0.060; visual mesh filename=package://assets/Module_right_front.stl
- link RH_SHOULDER: geometry collision box size=0.269 0.057 0.060; visual mesh filename=package://assets/Module_right_hind.stl
- link RH_UPPER_LEG: geometry collision box size=0.269 0.057 0.060; visual mesh filename=package://assets/Module_right_hind.stl
- link base_link: geometry collision box size=0.353 0.090 0.066; visual mesh filename=package://assets/Base.stl
- link body_left_F: geometry collision mesh filename=package://assets/body_left.stl; visual mesh filename=package://assets/body_left.stl
- link body_left_H: geometry collision mesh filename=package://assets/body_left.stl; visual mesh filename=package://assets/body_left.stl
- link body_right_F: geometry collision mesh filename=package://assets/body_right.stl; visual mesh filename=package://assets/body_right.stl
- link body_right_H: geometry collision mesh filename=package://assets/body_right.stl; visual mesh filename=package://assets/body_right.stl
- link wheel_1_LEFT_F: geometry collision mesh filename=package://assets/wheel.stl; visual mesh filename=package://assets/wheel.stl
- link wheel_1_LEFT_H: geometry collision mesh filename=package://assets/wheel.stl; visual mesh filename=package://assets/wheel.stl
- link wheel_1_RIGHT_F: geometry collision mesh filename=package://assets/wheel.stl; visual mesh filename=package://assets/wheel.stl
- link wheel_1_RIGHT_H: geometry collision mesh filename=package://assets/wheel.stl; visual mesh filename=package://assets/wheel.stl
- link wheel_2_LEFT_F: geometry collision mesh filename=package://assets/wheel.stl; visual mesh filename=package://assets/wheel.stl
- link wheel_2_LEFT_H: geometry collision mesh filename=package://assets/wheel.stl; visual mesh filename=package://assets/wheel.stl
- link wheel_2_RIGHT_F: geometry collision mesh filename=package://assets/wheel.stl; visual mesh filename=package://assets/wheel.stl
- link wheel_2_RIGHT_H: geometry collision mesh filename=package://assets/wheel.stl; visual mesh filename=package://assets/wheel.stl
- link wheel_3_LEFT_F: geometry collision mesh filename=package://assets/wheel.stl; visual mesh filename=package://assets/wheel.stl
- link wheel_3_LEFT_H: geometry collision mesh filename=package://assets/wheel.stl; visual mesh filename=package://assets/wheel.stl
- link wheel_3_RIGHT_F: geometry collision mesh filename=package://assets/wheel.stl; visual mesh filename=package://assets/wheel.stl
- link wheel_3_RIGHT_H: geometry collision mesh filename=package://assets/wheel.stl; visual mesh filename=package://assets/wheel.stl
- link wheel_4_LEFT_F: geometry collision mesh filename=package://assets/wheel.stl; visual mesh filename=package://assets/wheel.stl
- link wheel_4_LEFT_H: geometry collision mesh filename=package://assets/wheel.stl; visual mesh filename=package://assets/wheel.stl
- link wheel_4_RIGHT_F: geometry collision mesh filename=package://assets/wheel.stl; visual mesh filename=package://assets/wheel.stl
- link wheel_4_RIGHT_H: geometry collision mesh filename=package://assets/wheel.stl; visual mesh filename=package://assets/wheel.stl
