Commit message: change name of ankle joint in urdf

File: trackquad/urdf/traquad.urdf (robot description, URDF)
Before this commit: robot mulinex, 29 links, 28 joints
Joints:
- removed joint joint_left_F
- removed joint joint_left_H
- removed joint joint_right_F
- removed joint joint_right_H
- added joint LF_ANKLE: type revolute, parent LH_UPPER_LEG, child body_left_H, origin xyz=-0.19 0.05 0 rpy=1.5708 0 1.5708, axis 1 0 0, limit lower=-0.785398 upper=0.785398 effort=10 velocity=10
- added joint LH_ANKLE: type revolute, parent LF_UPPER_LEG, child body_left_F, origin xyz=0.19 0.05 0 rpy=-1.5708 0 1.5708, axis 1 0 0, limit lower=-0.785398 upper=0.785398 effort=10 velocity=10
- added joint RF_ANKLE: type revolute, parent RF_UPPER_LEG, child body_right_F, origin xyz=0.19 -0.05 0 rpy=3.14159 0 1.5708, axis 1 0 0, limit lower=-0.785398 upper=0.785398 effort=10 velocity=10
- added joint RH_ANKLE: type revolute, parent RH_UPPER_LEG, child body_right_H, origin xyz=-0.19 -0.05 0 rpy=0 0 1.5708, axis 1 0 0, limit lower=-0.785398 upper=0.785398 effort=10 velocity=10
